File: Hardware/Qwiic Shield for Arduino.sch (EAGLE design)
At the start: 21 parts, among them Q1 BSS138, Q2 BSS138, U1 ARDUINO UNO

Commit message: Changed over to Sparkfun library from SparkX
Parts:
- J1, J10, J8, J9: value (none) -> Qwiic Right Angle; device SparkX:I2C_STANDARDJS-1MM -> SparkFun-Connectors:I2C_STANDARDQWIIC
- U$2: value SPARKX-LOGO5 -> SFE_LOGO_NAME_FLAME.1_INCH; device SparkX:SPARKX-LOGO5 -> SparkFun-Aesthetics:SFE_LOGO_NAME_FLAME.1_INCH
Connections:
- net 3.3V: now also J1.2, J10.2, J8.2, J9.2; no longer J1.VCC, J10.VCC, J8.VCC, J9.VCC
- net GND: now also J1.1, J10.1, J8.1, J9.1; no longer J1.GND, J10.GND, J8.GND, J9.GND
- net SCL: now also J1.4, J10.4, J8.4, J9.4; no longer J1.SCL, J10.SCL, J8.SCL, J9.SCL
- net SDA: now also J1.3, J10.3, J8.3, J9.3; no longer J1.SDA, J10.SDA, J8.SDA, J9.SDA
Changed lines of the file:
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@@
 <part name="FD1" library="SparkFun-Aesthetics" deviceset="FIDUCIAL" device="1X2"/>
 <part name="FD2" library="SparkFun-Aesthetics" deviceset="FIDUCIAL" device="1X2"/>
-<part name="J1" library="SparkX" deviceset="I2C_STANDARD" device="JS-1MM"/>
+<part name="J1" library="SparkFun-Connectors" deviceset="I2C_STANDARD" device="QWIIC" value="Qwiic Right Angle"/>
 <part name="SUPPLY5" library="SparkFun-PowerSymbols" deviceset="3.3V" device=""/>
 <part name="SUPPLY6" library="SparkFun-PowerSymbols" deviceset="3.3V" device=""/>
@@
 <part name="SUPPLY8" library="SparkFun-PowerSymbols" deviceset="VIN" device=""/>
 <part name="SUPPLY10" library="SparkFun-PowerSymbols" deviceset="5V" device=""/>
-<part name="J8" library="SparkX" deviceset="I2C_STANDARD" device="JS-1MM"/>
+<part name="J8" library="SparkFun-Connectors" deviceset="I2C_STANDARD" device="QWIIC" value="Qwiic Right Angle"/>
 <part name="SUPPLY3" library="SparkFun-PowerSymbols" deviceset="3.3V" device=""/>
 <part name="GND5" library="SparkFun-PowerSymbols" deviceset="GND" device=""/>
-<part name="J9" library="SparkX" deviceset="I2C_STANDARD" device="JS-1MM"/>
+<part name="J9" library="SparkFun-Connectors" deviceset="I2C_STANDARD" device="QWIIC" value="Qwiic Right Angle"/>
 <part name="SUPPLY9" library="SparkFun-PowerSymbols" deviceset="3.3V" device=""/>
 <part name="GND6" library="SparkFun-PowerSymbols" deviceset="GND" device=""/>
-<part name="J10" library="SparkX" deviceset="I2C_STANDARD" device="JS-1MM"/>
+<part name="J10" library="SparkFun-Connectors" deviceset="I2C_STANDARD" device="QWIIC" value="Qwiic Right Angle"/>
 <part name="SUPPLY11" library="SparkFun-PowerSymbols" deviceset="3.3V" device=""/>
 <part name="GND7" library="SparkFun-PowerSymbols" deviceset="GND" device=""/>
-<part name="U$2" library="SparkX" deviceset="SPARKX-LOGO" device="5" value="SPARKX-LOGO5"/>
+<part name="U$2" library="SparkFun-Aesthetics" deviceset="SFE_LOGO_NAME_FLAME" device=".1_INCH" value="SFE_LOGO_NAME_FLAME.1_INCH"/>
 <part name="U$3" library="SparkX" deviceset="QWIIC_BOARD_OUTLINE" device="H"/>
 </parts>
@@
 <instance part="SUPPLY1" gate="G$1" x="78.74" y="142.24"/>
 <instance part="SUPPLY2" gate="G$1" x="78.74" y="109.22"/>
-<instance part="LOGO1" gate="G$1" x="134.62" y="10.16"/>
+<instance part="LOGO1" gate="G$1" x="218.44" y="45.72"/>
 <instance part="FD1" gate="G$1" x="241.3" y="30.48"/>
 <instance part="FD2" gate="G$1" x="246.38" y="30.48"/>
-<instance part="J1" gate="G$1" x="22.86" y="33.02" rot="MR180"/>
+<instance part="J1" gate="G$1" x="22.86" y="33.02" smashed="yes" rot="MR180">
+<attribute name="VALUE" x="42.926" y="17.78" size="1.778" layer="96" font="vector" rot="MR90" align="top-left"/>
+<attribute name="NAME" x="17.78" y="25.146" size="1.778" layer="95" font="vector" rot="MR180"/>
+</instance>
 <instance part="SUPPLY5" gate="G$1" x="35.56" y="38.1"/>
 <instance part="SUPPLY6" gate="G$1" x="63.5" y="109.22"/>
@@
 <instance part="SUPPLY8" gate="G$1" x="116.84" y="119.38"/>
 <instance part="SUPPLY10" gate="G$1" x="121.92" y="119.38"/>
-<instance part="J8" gate="G$1" x="53.34" y="33.02" rot="MR180"/>
+<instance part="J8" gate="G$1" x="53.34" y="33.02" smashed="yes" rot="MR180">
+<attribute name="VALUE" x="73.406" y="17.78" size="1.778" layer="96" font="vector" rot="MR90" align="top-left"/>
+<attribute name="NAME" x="48.26" y="25.146" size="1.778" layer="95" font="vector" rot="MR180"/>
+</instance>
 <instance part="SUPPLY3" gate="G$1" x="66.04" y="38.1"/>
 <instance part="GND5" gate="1" x="63.5" y="22.86"/>
-<instance part="J9" gate="G$1" x="83.82" y="33.02" rot="MR180"/>
+<instance part="J9" gate="G$1" x="83.82" y="33.02" smashed="yes" rot="MR180">
+<attribute name="VALUE" x="103.886" y="17.78" size="1.778" layer="96" font="vector" rot="MR90" align="top-left"/>
+<attribute name="NAME" x="78.74" y="25.146" size="1.778" layer="95" font="vector" rot="MR180"/>
+</instance>
 <instance part="SUPPLY9" gate="G$1" x="96.52" y="38.1"/>
 <instance part="GND6" gate="1" x="93.98" y="22.86"/>
-<instance part="J10" gate="G$1" x="114.3" y="33.02" rot="MR180"/>
+<instance part="J10" gate="G$1" x="114.3" y="33.02" smashed="yes" rot="MR180">
+<attribute name="VALUE" x="134.366" y="17.78" size="1.778" layer="96" font="vector" rot="MR90" align="top-left"/>
+<attribute name="NAME" x="109.22" y="25.146" size="1.778" layer="95" font="vector" rot="MR180"/>
+</instance>
 <instance part="SUPPLY11" gate="G$1" x="127" y="38.1"/>
 <instance part="GND7" gate="1" x="124.46" y="22.86"/>
-<instance part="U$2" gate="G$1" x="106.68" y="7.62"/>
-<instance part="U$3" gate="G$1" x="83.82" y="7.62"/>
+<instance part="U$2" gate="G$1" x="147.32" y="35.56"/>
+<instance part="U$3" gate="G$1" x="241.3" y="40.64"/>
 </instances>
 <busses>
@@
 </segment>
 <segment>
-<pinref part="J1" gate="G$1" pin="GND"/>
+<pinref part="J1" gate="G$1" pin="1"/>
 <wire x1="30.48" y1="35.56" x2="33.02" y2="35.56" width="0.1524" layer="91"/>
 <wire x1="33.02" y1="35.56" x2="33.02" y2="25.4" width="0.1524" layer="91"/>
@@
 </segment>
 <segment>
-<pinref part="J8" gate="G$1" pin="GND"/>
+<pinref part="J8" gate="G$1" pin="1"/>
 <wire x1="60.96" y1="35.56" x2="63.5" y2="35.56" width="0.1524" layer="91"/>
 <wire x1="63.5" y1="35.56" x2="63.5" y2="25.4" width="0.1524" layer="91"/>
@@
 </segment>
 <segment>
-<pinref part="J9" gate="G$1" pin="GND"/>
+<pinref part="J9" gate="G$1" pin="1"/>
 <wire x1="91.44" y1="35.56" x2="93.98" y2="35.56" width="0.1524" layer="91"/>
 <wire x1="93.98" y1="35.56" x2="93.98" y2="25.4" width="0.1524" layer="91"/>
@@
 </segment>
 <segment>
-<pinref part="J10" gate="G$1" pin="GND"/>
+<pinref part="J10" gate="G$1" pin="1"/>
 <wire x1="121.92" y1="35.56" x2="124.46" y2="35.56" width="0.1524" layer="91"/>
 <wire x1="124.46" y1="35.56" x2="124.46" y2="25.4" width="0.1524" layer="91"/>
@@
 <net name="3.3V" class="0">
 <segment>
-<pinref part="J1" gate="G$1" pin="VCC"/>
+<pinref part="J1" gate="G$1" pin="2"/>
 <wire x1="30.48" y1="33.02" x2="35.56" y2="33.02" width="0.1524" layer="91"/>
 <wire x1="35.56" y1="33.02" x2="35.56" y2="38.1" width="0.1524" layer="91"/>
@@
 </segment>
 <segment>
-<pinref part="J8" gate="G$1" pin="VCC"/>
+<pinref part="J8" gate="G$1" pin="2"/>
 <wire x1="60.96" y1="33.02" x2="66.04" y2="33.02" width="0.1524" layer="91"/>
 <wire x1="66.04" y1="33.02" x2="66.04" y2="38.1" width="0.1524" layer="91"/>
@@
 </segment>
 <segment>
-<pinref part="J9" gate="G$1" pin="VCC"/>
+<pinref part="J9" gate="G$1" pin="2"/>
 <wire x1="91.44" y1="33.02" x2="96.52" y2="33.02" width="0.1524" layer="91"/>
 <wire x1="96.52" y1="33.02" x2="96.52" y2="38.1" width="0.1524" layer="91"/>
@@
 </segment>
 <segment>
-<pinref part="J10" gate="G$1" pin="VCC"/>
+<pinref part="J10" gate="G$1" pin="2"/>
 <wire x1="121.92" y1="33.02" x2="127" y2="33.02" width="0.1524" layer="91"/>
 <wire x1="127" y1="33.02" x2="127" y2="38.1" width="0.1524" layer="91"/>
@@
 </segment>
 <segment>
-<pinref part="J1" gate="G$1" pin="SCL"/>
+<pinref part="J1" gate="G$1" pin="4"/>
 <wire x1="30.48" y1="27.94" x2="35.56" y2="27.94" width="0.1524" layer="91"/>
 <label x="35.56" y="27.94" size="1.27" layer="95" xref="yes"/>
 </segment>
 <segment>
-<pinref part="J8" gate="G$1" pin="SCL"/>
+<pinref part="J8" gate="G$1" pin="4"/>
 <wire x1="60.96" y1="27.94" x2="66.04" y2="27.94" width="0.1524" layer="91"/>
 <label x="66.04" y="27.94" size="1.27" layer="95" xref="yes"/>
 </segment>
 <segment>
-<pinref part="J9" gate="G$1" pin="SCL"/>
+<pinref part="J9" gate="G$1" pin="4"/>
 <wire x1="91.44" y1="27.94" x2="96.52" y2="27.94" width="0.1524" layer="91"/>
 <label x="96.52" y="27.94" size="1.27" layer="95" xref="yes"/>
 </segment>
 <segment>
-<pinref part="J10" gate="G$1" pin="SCL"/>
+<pinref part="J10" gate="G$1" pin="4"/>
 <wire x1="121.92" y1="27.94" x2="127" y2="27.94" width="0.1524" layer="91"/>
 <label x="127" y="27.94" size="1.27" layer="95" xref="yes"/>
@@
 </segment>
 <segment>
-<pinref part="J1" gate="G$1" pin="SDA"/>
+<pinref part="J1" gate="G$1" pin="3"/>
 <wire x1="30.48" y1="30.48" x2="35.56" y2="30.48" width="0.1524" layer="91"/>
 <label x="35.56" y="30.48" size="1.27" layer="95" xref="yes"/>
 </segment>
 <segment>
-<pinref part="J8" gate="G$1" pin="SDA"/>
+<pinref part="J8" gate="G$1" pin="3"/>
 <wire x1="60.96" y1="30.48" x2="66.04" y2="30.48" width="0.1524" layer="91"/>
 <label x="66.04" y="30.48" size="1.27" layer="95" xref="yes"/>
 </segment>
 <segment>
-<pinref part="J9" gate="G$1" pin="SDA"/>
+<pinref part="J9" gate="G$1" pin="3"/>
 <wire x1="91.44" y1="30.48" x2="96.52" y2="30.48" width="0.1524" layer="91"/>
 <label x="96.52" y="30.48" size="1.27" layer="95" xref="yes"/>
 </segment>
 <segment>
-<pinref part="J10" gate="G$1" pin="SDA"/>
+<pinref part="J10" gate="G$1" pin="3"/>
 <wire x1="121.92" y1="30.48" x2="127" y2="30.48" width="0.1524" layer="91"/>
 <label x="127" y="30.48" size="1.27" layer="95" xref="yes"/>

Commit message: Partially completed checklist, changes still need to be made
Parts:
- added LOGO2: REVISION, SparkFun-Aesthetics:REVISION
Other:
- note added: "Andrew England"
- note added: "V01"
- note removed: "X11"
- moved on the sheet: J2, J3, J4, J6, Q1, Q2, R2, R3, R4, R5, U1

Commit message: Completed checklist + pre-design review changes
Parts:
- added FD3, FD4: FIDUCIAL1X2, SparkFun-Aesthetics:FIDUCIAL1X2
Changed lines of the file:
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@@
 <part name="U$3" library="SparkX" deviceset="QWIIC_BOARD_OUTLINE" device="H"/>
 <part name="LOGO2" library="SparkFun-Aesthetics" deviceset="REVISION" device=""/>
+<part name="FD3" library="SparkFun-Aesthetics" deviceset="FIDUCIAL" device="1X2"/>
+<part name="FD4" library="SparkFun-Aesthetics" deviceset="FIDUCIAL" device="1X2"/>
 </parts>
 <sheets>
@@
 <instance part="U$3" gate="G$1" x="241.3" y="40.64"/>
 <instance part="LOGO2" gate="G$1" x="148.59" y="6.858"/>
+<instance part="FD3" gate="G$1" x="243.84" y="30.48"/>
+<instance part="FD4" gate="G$1" x="238.76" y="30.48"/>
 </instances>
 <busses>

Commit message: Changed version number
Other:
- note added: "V10"
- note removed: "V01"
Changed lines of the file:
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@@
 Conversion</text>
 <text x="170.18" y="154.94" size="3.048" layer="97" font="vector" ratio="12">Arduino</text>
-<text x="236.22" y="7.62" size="2.54" layer="94" font="vector">V01</text>
+<text x="236.22" y="7.62" size="2.54" layer="94" font="vector">V10</text>
 <text x="38.1" y="45.72" size="3.048" layer="97" font="vector" ratio="12">I2C Connectors</text>
 <text x="168.656" y="6.858" size="2.54" layer="94" font="vector">Andrew England</text>

Commit message: Connected R3 SDA/SCL pins and IOREF
-SDA and SCL are now connected to both A4 /A5 pins and SDA/SCL pins.
-Changed "high" logic side of converters to IOREF, to allow the Arduino to supply it's own IOREF. This will allow the shield to work with 3.3V logic Arduinos.
-named PTH headers in the row of 3.3V to avoid overlap DRC errors.
bumped version to v11 insch and brd
- Added I2C pullup jumper to bottom side with label
- rerouted SDA/SCL to allow for better GND return in pour
- bumped up 3.3V traces to 0.020 inch for qwiic connectors
- all labels to buzzrds and included qwiic logo
Parts:
- removed R5: 4.7K, SparkFun-Resistors:4.7KOHM-1/10W-1%(0603)
- added I2C: JUMPER-SMT_3_2-NC_TRACE_SILK, SparkFun-Jumpers:JUMPER-SMT_3_2-NC_TRACE_SILK
- added LOGO3: QWIIC_LOGO_6MM, SparkFun-Aesthetics:QWIIC_LOGO_6MM
- added R1: 4.7k, SparkFun-Resistors:4.7KOHM-0603-1/10W-1%
- R2: value 4.7K -> 4.7k; device SparkFun-Resistors:4.7KOHM-1/10W-1%(0603) -> SparkFun-Resistors:4.7KOHM-0603-1/10W-1%
Connections:
- removed net HV_SCL: J4.1, Q2.D, R5.2, U1.A5
- removed net HV_SDA: J4.2, Q1.D, R4.2, U1.A4
- removed net SCL1: J3.10, U1.SCL
- removed net SDA1: J3.9, U1.SDA
- new net N$76: I2C.3, R1.2
- new net N$78: I2C.1, R2.2
- new net SCL_R3: J3.10, J4.1, Q2.D, R3.2, U1.A5, U1.SCL
- new net SDA_R3: J3.9, J4.2, Q1.D, R4.2, U1.A4, U1.SDA
- net 3.3V: now also I2C.2; no longer R2.1, R3.1
- net 5V: no longer R4.1, R5.1
- net IOREF: now also R3.1, R4.1
- net SCL: now also R2.1; no longer R2.2
- net SDA: now also R1.1; no longer R3.2
Other:
- note added: "Andrew England, Pete Lewis"
- note added: "Cut this jumper to remove 4.7k pull-up resistors."
- note added: "V11"
- note removed: "Andrew England"
- note removed: "V10"
- moved on the sheet: J2, J3, J4, J6, Q1, Q2, R2, R3, R4, U1

Commit message: Moved qwiic board to SFE library
Parts:
- U$3: device SparkX:QWIIC_BOARD_OUTLINEH -> SparkFun-Boards:QWIIC_BOARD_OUTLINEH
Changed lines of the file:
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@@
 <part name="GND7" library="SparkFun-PowerSymbols" deviceset="GND" device=""/>
 <part name="U$2" library="SparkFun-Aesthetics" deviceset="SFE_LOGO_NAME_FLAME" device=".1_INCH" value="SFE_LOGO_NAME_FLAME.1_INCH"/>
-<part name="U$3" library="SparkX" deviceset="QWIIC_BOARD_OUTLINE" device="H"/>
+<part name="U$3" library="SparkFun-Boards" deviceset="QWIIC_BOARD_OUTLINE" device="H"/>
 <part name="LOGO2" library="SparkFun-Aesthetics" deviceset="REVISION" device=""/>
 <part name="FD3" library="SparkFun-Aesthetics" deviceset="FIDUCIAL" device="1X2"/>
